File: FIRST_BLOCK.kicad_sch (KiCad schematic)
At the start: 14 parts, among them Q1 IRF540N, Q2 IRF540N, U2 IR2110S

Commit message: Layout almost done..
Parts:
- removed C3: 22uF, Capacitor_THT:CP_Radial_D8.0mm_P3.80mm, symbol Device:C_Small_US
- C6: footprint Capacitor_THT:CP_Radial_D8.0mm_P3.80mm -> Capacitor_THT:CP_Radial_D5.0mm_P2.50mm
- R1, R2, R3, R4: footprint Resistor_THT:R_Axial_DIN0309_L9.0mm_D3.2mm_P12.70mm_Horizontal -> Resistor_THT:R_Axial_DIN0207_L6.3mm_D2.5mm_P10.16mm_Horizontal
Other:
- moved on the sheet: C4, C5, C6, D2, D3, D4, Q1, Q2, R1, R2, R3, R4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
