File: THIRD_BLOCK.kicad_sch (KiCad schematic)
At the start: 14 parts, among them Q5 IRF540N, Q6 IRF540N, U4 IR2110S

Commit message: Layout almost done..
Parts:
- removed C11: 22uF, Capacitor_THT:CP_Radial_D8.0mm_P3.80mm, symbol Device:C_Small_US
- R10, R11, R12, R9: footprint Resistor_THT:R_Axial_DIN0309_L9.0mm_D3.2mm_P12.70mm_Horizontal -> Resistor_THT:R_Axial_DIN0207_L6.3mm_D2.5mm_P10.16mm_Horizontal
- renumbered C12 to C10, C13 to C11, C14 to C12
Changed lines of the file:
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@@
-	)
-	(junction
-		(at 99.06 54.61)
-		(diameter 0)
-		(color 0 0 0 0)
 	)
 	(junction
@@
 		(color 0 0 0 0)
 	)
-	(junction
-		(at 92.71 66.04)
-		(diameter 0)
-		(color 0 0 0 0)
-	)
 	(wire
 		(pts
@@
 	(wire
 		(pts
-			(xy 87.63 54.61) (xy 87.63 57.15)
-		)
-		(stroke
-			(width 0)
-			(type default)
-		)
-	)
-	(wire
-		(pts
 			(xy 116.84 90.17) (xy 116.84 95.25)
 		)
@@
 	(wire
 		(pts
-			(xy 92.71 66.04) (xy 99.06 66.04)
-		)
-		(stroke
-			(width 0)
-			(type default)
-		)
-	)
-	(wire
-		(pts
 			(xy 127 86.36) (xy 175.26 86.36)
 		)
@@
 	(wire
 		(pts
-			(xy 99.06 54.61) (xy 87.63 54.61)
-		)
-		(stroke
-			(width 0)
-			(type default)
-		)
-	)
-	(wire
-		(pts
-			(xy 87.63 66.04) (xy 92.71 66.04)
-		)
-		(stroke
-			(width 0)
-			(type default)
-		)
-	)
-	(wire
-		(pts
-			(xy 87.63 62.23) (xy 87.63 66.04)
-		)
-		(stroke
-			(width 0)
-			(type default)
-		)
-	)
-	(wire
-		(pts
-			(xy 92.71 66.04) (xy 92.71 67.31)
-		)
-		(stroke
-			(width 0)
-			(type default)
-		)
-	)
-	(wire
-		(pts
 			(xy 119.38 54.61) (xy 99.06 54.61)
 		)
@@
 	(wire
 		(pts
-			(xy 99.06 66.04) (xy 99.06 62.23)
+			(xy 99.06 62.23) (xy 99.06 67.31)
 		)
 		(stroke
@@
 			)
 		)
-		(property "Footprint" "Resistor_THT:R_Axial_DIN0309_L9.0mm_D3.2mm_P12.70mm_Horizontal"
+		(property "Footprint" "Resistor_THT:R_Axial_DIN0207_L6.3mm_D2.5mm_P10.16mm_Horizontal"
 			(at 182.88 72.39 0)
 			(effects
@@
 		(dnp no)
 		(fields_autoplaced yes)
-		(property "Reference" "C14"
+		(property "Reference" "C12"
 			(at 165.1 74.8029 0)
 			(effects
@@
 			(project "Motror driver"
 				(path "/07601b07-483c-472d-8aca-89f8ac7b9045/2f0f577d-d655-4c5f-83ab-c4a2664c8dfc"
-					(reference "C14")
+					(reference "C12")
 					(unit 1)
 				)
@@
 		(on_board yes)
 		(dnp no)
-		(property "Reference" "C12"
+		(property "Reference" "C10"
 			(at 101.6 58.4262 0)
 			(effects
@@
 			(project "Motror driver"
 				(path "/07601b07-483c-472d-8aca-89f8ac7b9045/2f0f577d-d655-4c5f-83ab-c4a2664c8dfc"
-					(reference "C12")
+					(reference "C10")
 					(unit 1)
 				)
@@
 	(symbol
 		(lib_id "power:GND")
-		(at 92.71 67.31 0)
+		(at 99.06 67.31 0)
 		(unit 1)
 		(exclude_from_sim no)
@@
 		(fields_autoplaced yes)
 		(property "Reference" "#PWR018"
-			(at 92.71 73.66 0)
+			(at 99.06 73.66 0)
 			(effects
 				(font
@@
 		)
 		(property "Value" "GND"
-			(at 92.71 72.39 0)
+			(at 99.06 72.39 0)
 			(effects
 				(font
@@
 		)
 		(property "Footprint" ""
-			(at 92.71 67.31 0)
+			(at 99.06 67.31 0)
 			(effects
 				(font
@@
 		)
 		(property "Datasheet" ""
-			(at 92.71 67.31 0)
+			(at 99.06 67.31 0)
 			(effects
 				(font
@@
 		)
 		(property "Description" "Power symbol creates a global label with name \"GND\" , ground"
-			(at 92.71 67.31 0)
+			(at 99.06 67.31 0)
 			(effects
 				(font
@@
 	)
 	(symbol
-		(lib_id "Device:C_Small_US")
-		(at 87.63 59.69 0)
-		(unit 1)
-		(exclude_from_sim no)
-		(in_bom yes)
-		(on_board yes)
-		(dnp no)
-		(fields_autoplaced yes)
-		(property "Reference" "C11"
-			(at 90.17 58.5469 0)
-			(effects
-				(font
-					(size 1.27 1.27)
-				)
-				(justify left)
-			)
-		)
-		(property "Value" "22uF"
-			(at 90.17 61.0869 0)
-			(effects
-				(font
-					(size 1.27 1.27)
-				)
-				(justify left)
-			)
-		)
-		(property "Footprint" "Capacitor_THT:CP_Radial_D8.0mm_P3.80mm"
-			(at 87.63 59.69 0)
-			(effects
-				(font
-					(size 1.27 1.27)
-				)
-				(hide yes)
-			)
-		)
-		(property "Datasheet" ""
-			(at 87.63 59.69 0)
-			(effects
-				(font
-					(size 1.27 1.27)
-				)
-				(hide yes)
-			)
-		)
-		(property "Description" "capacitor, small US symbol"
-			(at 87.63 59.69 0)
-			(effects
-				(font
-					(size 1.27 1.27)
-				)
-				(hide yes)
-			)
-		)
-		(pin "1"
-		)
-		(pin "2"
-		)
-		(instances
-			(project "Motror driver"
-				(path "/07601b07-483c-472d-8aca-89f8ac7b9045/2f0f577d-d655-4c5f-83ab-c4a2664c8dfc"
-					(reference "C11")
-					(unit 1)
-				)
-			)
-		)
-	)
-	(symbol
 		(lib_id "Diode:1N4007")
 		(at 138.43 82.55 180)
@@
 			)
 		)
-		(property "Footprint" "Resistor_THT:R_Axial_DIN0309_L9.0mm_D3.2mm_P12.70mm_Horizontal"
+		(property "Footprint" "Resistor_THT:R_Axial_DIN0207_L6.3mm_D2.5mm_P10.16mm_Horizontal"
 			(at 182.88 86.36 0)
 			(effects
@@
 		(on_board yes)
 		(dnp no)
-		(property "Reference" "C13"
+		(property "Reference" "C11"
 			(at 152.4 77.4638 0)
 			(effects
@@
 			(project "Motror driver"
 				(path "/07601b07-483c-472d-8aca-89f8ac7b9045/2f0f577d-d655-4c5f-83ab-c4a2664c8dfc"
-					(reference "C13")
+					(reference "C11")
 					(unit 1)
 				)
@@
 			)
 		)
-		(property "Footprint" "Resistor_THT:R_Axial_DIN0309_L9.0mm_D3.2mm_P12.70mm_Horizontal"
+		(property "Footprint" "Resistor_THT:R_Axial_DIN0207_L6.3mm_D2.5mm_P10.16mm_Horizontal"
 			(at 200.66 91.44 0)
 			(effects
@@
 			)
 		)
-		(property "Footprint" "Resistor_THT:R_Axial_DIN0309_L9.0mm_D3.2mm_P12.70mm_Horizontal"
+		(property "Footprint" "Resistor_THT:R_Axial_DIN0207_L6.3mm_D2.5mm_P10.16mm_Horizontal"
 			(at 200.66 76.2 0)
 			(effects
