File: MotorIO.kicad_pcb (KiCad board)
At the start: 2 copper layers, 50 parts, among them J1 Conn_01x02_Pin, J2 Conn_01x02_Pin, J3 Conn_01x09, J4 Conn_01x03_Pin, Q1 IRF540N, Q2 IRF540N, Q3 IRF540N, Q4 IRF540N, Q5 IRF540N, Q6 IRF540N, U1 AMS1117-3.3, U2 IR2110S, U3 IR2110S, U4 IR2110S

Commit message: Layout almost done..
Parts:
- removed C13: 100nF, Capacitor_THT:C_Disc_D3.8mm_W2.6mm_P2.50mm
- removed C14: 22uF, Capacitor_THT:CP_Radial_D8.0mm_P3.80mm
- removed J3: Conn_01x09, Connector_PinHeader_2.54mm:PinHeader_1x09_P2.54mm_Vertical
- removed J4: Conn_01x03_Pin, Connector_PinSocket_2.54mm:PinSocket_1x03_P2.54mm_Vertical
- added H1: MountingHole, MountingHole:MountingHole_2.2mm_M2_DIN965, F.Cu at (105.3, 51.4)
- added H2: MountingHole, MountingHole:MountingHole_2.2mm_M2_DIN965, F.Cu at (170.3, 51.4)
- added H3: MountingHole, MountingHole:MountingHole_2.2mm_M2_DIN965, F.Cu at (170.3, 137.8)
- added H4: MountingHole, MountingHole:MountingHole_2.2mm_M2_DIN965, F.Cu at (105.3, 137.8)
- added J5: Barrel_Jack_Switch, Connector_BarrelJack:BarrelJack_Kycon_KLDX-0202-xC_Horizontal, F.Cu at (115.8, 57.5)
- added J6: Screw_Terminal_01x03, TerminalBlock_Phoenix:TerminalBlock_Phoenix_MKDS-1,5-3_1x03_P5.00mm_Horizontal, F.Cu at (115.1, 105.3)
- added J7: Screw_Terminal_01x09, TerminalBlock_Phoenix:TerminalBlock_Phoenix_MKDS-1,5-9_1x09_P5.00mm_Horizontal, F.Cu at (164.3, 127.8)
- C10, C11, C7: value 22uF -> 100nF; footprint Capacitor_THT:CP_Radial_D8.0mm_P3.80mm -> Capacitor_THT:C_Disc_D3.8mm_W2.6mm_P2.50mm
- C12, C9: value 100nF -> 22uF; footprint Capacitor_THT:C_Disc_D3.8mm_W2.6mm_P2.50mm -> Capacitor_THT:CP_Radial_D5.0mm_P2.50mm
- C3: value 22uF -> 100uF; footprint Capacitor_THT:CP_Radial_D8.0mm_P3.80mm -> Capacitor_THT:CP_Radial_D10.0mm_P5.00mm
- C6: footprint Capacitor_THT:CP_Radial_D8.0mm_P3.80mm -> Capacitor_THT:CP_Radial_D5.0mm_P2.50mm
- R1, R10, R11, R12, R2, R3, R4, R5, R6, R7, R8, R9: footprint Resistor_THT:R_Axial_DIN0309_L9.0mm_D3.2mm_P12.70mm_Horizontal -> Resistor_THT:R_Axial_DIN0207_L6.3mm_D2.5mm_P10.16mm_Horizontal
- moved R11 107.4 mm to (147.5, 139.3), turned to 90 degrees
- moved Q5 97.9 mm to (153.0, 130.7), turned to -90 degrees
- moved R9 97.1 mm to (129.8, 133.8)
- moved R12 96.9 mm to (148.0, 124.8), turned to 90 degrees
- moved C11 93.9 mm to (126.3, 126.6), turned to -90 degrees
- moved C10 89.7 mm to (143.3, 127.1), turned to 90 degrees
- moved C7 87.9 mm to (143.6, 96.6), turned to 90 degrees
- moved R8 85.8 mm to (148.2, 94.3), turned to 90 degrees
- moved Q6 85.8 mm to (153.0, 117.2), turned to -90 degrees
- moved D9 84.6 mm to (129.9, 138.7)
- moved R7 83.9 mm to (147.7, 108.8), turned to 90 degrees
- moved R10 83.1 mm to (130.1, 117.3)
- moved C12 81.1 mm to (121.3, 126.7), turned to -90 degrees
- moved D7 77.8 mm to (130.3, 82.4)
- moved C8 74.8 mm to (126.6, 96.1), turned to -90 degrees
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Connections:
- C10 pad 1: /Phase2/OUT2 -> +3.3V
- C10 pad 2: Net-(D5-K) -> GND
- C11 pad 1: +3.3V -> /Phase3/OUT1
- C11 pad 2: GND -> Net-(D8-K)
- C12 pad 1: +3.3V -> /Phase3/OUT1
- C12 pad 2: GND -> Net-(D8-K)
- C8 pad 1: +3.3V -> /Phase2/OUT1
- C8 pad 2: GND -> Net-(D5-K)
- C9 pad 1: /Phase2/OUT2 -> /Phase2/OUT1
- Q3 pad 3: /Phase2/OUT2 -> /Phase2/OUT1
- Q4 pad 2: /Phase2/OUT2 -> /Phase2/OUT1
- Q5 pad 3: /Phase3/OUT3 -> /Phase3/OUT1
- Q6 pad 2: /Phase3/OUT3 -> /Phase3/OUT1
- R11 pad 1: /Phase3/OUT3 -> /Phase3/OUT1
- R7 pad 1: /Phase2/OUT2 -> /Phase2/OUT1
- U3 pad 12: /Phase2/HIN2 -> /Phase2/HIN1
- U3 pad 14: /Phase2/LIN2 -> /Phase2/LIN1
- U3 pad 6: /Phase2/OUT2 -> /Phase2/OUT1
- U4 pad 12: /Phase3/HIN3 -> /Phase3/HIN1
- U4 pad 14: /Phase3/LIN3 -> /Phase3/LIN1
- U4 pad 6: /Phase3/OUT3 -> /Phase3/OUT1
Routing:
- net +12V: track 0.00 -> 351.3 mm
- net /Phase2/OUT1: track 0.00 -> 148.8 mm
- net /Phase3/OUT1: track 0.00 -> 136.3 mm, vias 0 -> 1
- net +3.3V: track 0.00 -> 132.6 mm, vias 0 -> 3
- net /Phase1/OUT1: track 0.00 -> 121.1 mm, vias 0 -> 1
- net GND: track 0.00 -> 63.5 mm, vias 0 -> 15
- net /Phase1/HIN1: track 0.00 -> 63.0 mm, vias 0 -> 2
- net Net-(D6-A): track 0.00 -> 62.0 mm
- net Net-(D9-A): track 0.00 -> 62.0 mm
- net Net-(D7-A): track 0.00 -> 57.2 mm
- net Net-(D10-A): track 0.00 -> 57.2 mm
- net /Phase1/LIN1: track 0.00 -> 56.7 mm, vias 0 -> 2
- net Net-(D8-K): track 0.00 -> 45.0 mm
- net Net-(D5-K): track 0.00 -> 45.0 mm
- net /Phase2/HIN1: track 0.00 -> 41.6 mm, vias 0 -> 1
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- added copper zone on F.Cu, net +3.3V
- added copper zone on B.Cu, net GND
Other:
- board outline added: 71.8 x 94.5 mm

Commit message: Layout done..
Parts:
- removed J7: Screw_Terminal_01x09, TerminalBlock_Phoenix:TerminalBlock_Phoenix_MKDS-1,5-9_1x09_P5.00mm_Horizontal
- added J3: MOTOR INPUTS, Connector_PinHeader_2.54mm:PinHeader_1x07_P2.54mm_Vertical, F.Cu at (166.8, 96.8)
- added kibuzzard-6931A7DA: G***, kibuzzard-6931A7DA, F.Cu at (134.3, 51.9)
- added kibuzzard-6931A81E: G***, kibuzzard-6931A81E, F.Cu at (127.3, 50.4)
- added kibuzzard-6931A834: G***, kibuzzard-6931A834, F.Cu at (127.3, 53.9)
- added kibuzzard-6931A882: G***, kibuzzard-6931A882, F.Cu at (170.6, 112.1)
- added kibuzzard-6931A8E0: G***, kibuzzard-6931A8E0, F.Cu at (170.6, 96.8)
- added kibuzzard-6931A8F1: G***, kibuzzard-6931A8F1, F.Cu at (170.6, 99.3)
- added kibuzzard-6931A900: G***, kibuzzard-6931A900, F.Cu at (170.6, 102.1)
- added kibuzzard-6931A90C: G***, kibuzzard-6931A90C, F.Cu at (170.6, 104.3)
- added kibuzzard-6931A916: G***, kibuzzard-6931A916, F.Cu at (170.6, 106.8)
- added kibuzzard-6931A91E: G***, kibuzzard-6931A91E, F.Cu at (170.6, 109.6)
- added kibuzzard-6931AA34: G***, kibuzzard-6931AA34, F.Cu at (105.3, 104.8)
- added kibuzzard-6931AA3C: G***, kibuzzard-6931AA3C, F.Cu at (105.3, 109.8)
- added kibuzzard-6931AA45: G***, kibuzzard-6931AA45, F.Cu at (105.3, 114.8)
- J1: value Conn_01x02_Pin -> POWER INPUTS
- J2: value Conn_01x02_Pin -> GND PINS
- J6: value Screw_Terminal_01x03 -> MOTOR OUTPUT
- moved J6 2.87 mm to (112.3, 104.8)
- moved D9 1.35 mm to (129.9, 137.3)
- moved J1 1.00 mm to (123.3, 50.6)
- moved J2 1.00 mm to (131.3, 53.1)
Routing:
- net /Phase3/HIN1: track 34.0 -> 51.6 mm
- net Net-(D9-K): track 27.6 -> 16.3 mm
- net Net-(D9-A): track 62.0 -> 50.7 mm
- net /Phase2/OUT1: track 148.8 -> 137.8 mm
- net /Phase3/LIN1: track 27.9 -> 36.8 mm
- net /Phase3/OUT1: track 136.3 -> 128.8 mm
- net /Phase1/LIN1: track 56.7 -> 63.0 mm
- net +12V: track 351.3 -> 357.2 mm
- net /Phase1/HIN1: track 63.0 -> 68.3 mm
- net /Phase1/OUT1: track 121.1 -> 122.8 mm
- net /Phase2/HIN1: track 41.6 -> 40.3 mm
- added copper zone on F.Cu, net GND
