File: MotorIO.kicad_sch (KiCad schematic)
At the start: 8 parts, among them J1 Conn_01x02_Pin, J2 Conn_01x02_Pin, J3 Conn_01x09, J4 Conn_01x03_Pin, U1 AMS1117-3.3

Commit message: Layout almost done..
Parts:
- removed J3: Conn_01x09, Connector_PinHeader_2.54mm:PinHeader_1x09_P2.54mm_Vertical, symbol Connector_Generic:Conn_01x09
- removed J4: Conn_01x03_Pin, Connector_PinSocket_2.54mm:PinSocket_1x03_P2.54mm_Vertical, symbol Connector:Conn_01x03_Pin
- added C3: 100uF, Capacitor_THT:CP_Radial_D10.0mm_P5.00mm, symbol Device:C_Small_US
- added H1, H2, H3, H4: MountingHole, MountingHole:MountingHole_2.2mm_M2_DIN965, symbol Mechanical:MountingHole
- added J5: Barrel_Jack_Switch, Connector_BarrelJack:BarrelJack_Kycon_KLDX-0202-xC_Horizontal, symbol Connector:Barrel_Jack_Switch
- added J6: Screw_Terminal_01x03, TerminalBlock_Phoenix:TerminalBlock_Phoenix_MKDS-1,5-3_1x03_P5.00mm_Horizontal, symbol Connector:Screw_Terminal_01x03
- added J7: Screw_Terminal_01x09, TerminalBlock_Phoenix:TerminalBlock_Phoenix_MKDS-1,5-9_1x09_P5.00mm_Horizontal, symbol Connector:Screw_Terminal_01x09
Connections:
- net +12V: now also J5.1
- net +3.3V: now also C3.1
- net GND: now also C3.2, J5.2, J5.3, J7.1 (Pin_1), J7.4 (Pin_4), J7.7 (Pin_7)
- net Phase1/HIN1: now also J7.8 (Pin_8)
- net Phase1/LIN1: now also J7.9 (Pin_9)
- net Phase1/OUT1: now also J6.1 (Pin_1)
- new net Phase2/HIN1: J7.5 (Pin_5)
- new net Phase2/LIN1: J7.6 (Pin_6)
- new net Phase2/OUT1: J6.2 (Pin_2)
- new net Phase3/HIN1: J7.2 (Pin_2)
- new net Phase3/LIN1: J7.3 (Pin_3)
- new net Phase3/OUT1: J6.3 (Pin_3)
Other:
- sheet Phase2: file SECOND_BLOCK.kicad_sch -> FIRST_BLOCK.kicad_sch
- sheet Phase2 ports: added HIN1, LIN1, OUT1; removed HIN2, LIN2, OUT2
- sheet Phase3: file THIRD_BLOCK.kicad_sch -> FIRST_BLOCK.kicad_sch
- sheet Phase3 ports: added HIN1, LIN1, OUT1; removed HIN3, LIN3, OUT3

Commit message: Layout done..
Parts:
- removed J7: Screw_Terminal_01x09, TerminalBlock_Phoenix:TerminalBlock_Phoenix_MKDS-1,5-9_1x09_P5.00mm_Horizontal, symbol Connector:Screw_Terminal_01x09
- added J3: MOTOR INPUTS, Connector_PinHeader_2.54mm:PinHeader_1x07_P2.54mm_Vertical, symbol Connector:Conn_01x07_Pin
- J1: value Conn_01x02_Pin -> POWER INPUTS
- J2: value Conn_01x02_Pin -> GND PINS
- J6: value Screw_Terminal_01x03 -> MOTOR OUTPUT
Connections:
- net GND: now also J3.7 (Pin_7)
- net Phase1/HIN1: now also J3.2 (Pin_2)
- net Phase1/LIN1: now also J3.1 (Pin_1)
- net Phase2/HIN1: now also J3.4 (Pin_4)
- net Phase2/LIN1: now also J3.3 (Pin_3)
- net Phase3/HIN1: now also J3.6 (Pin_6)
- net Phase3/LIN1: now also J3.5 (Pin_5)
